Commit message: walk benchmark envs

File: assets/urdf/go1/urdf/go1.urdf (robot description, URDF)
Before this commit: robot go1_description, 23 links, 22 joints
Links:
- link FL_calf: geometry collision box size=0.213 0.016 0.016
- link FL_foot: geometry collision sphere radius=0.02
- link FL_hip: geometry collision cylinder length=0.04 radius=0.046
- link FL_thigh: geometry collision box size=0.213 0.0245 0.034
- link FR_calf: geometry collision box size=0.213 0.016 0.016
- link FR_foot: geometry collision sphere radius=0.02
- link FR_hip: geometry collision cylinder length=0.04 radius=0.046
- link FR_thigh: geometry collision box size=0.213 0.0245 0.034
- link RL_calf: geometry collision box size=0.213 0.016 0.016
- link RL_foot: geometry collision sphere radius=0.02
- link RL_hip: geometry collision cylinder length=0.04 radius=0.046
- link RL_thigh: geometry collision box size=0.213 0.0245 0.034
- link RR_calf: geometry collision box size=0.213 0.016 0.016
- link RR_foot: geometry collision sphere radius=0.02
- link RR_hip: geometry collision cylinder length=0.04 radius=0.046
- link RR_thigh: geometry collision box size=0.213 0.0245 0.034
- link base: geometry 
- link imu_link: geometry 
- link trunk: geometry collision box size=0.3762 0.0935 0.114
