Commit message: add 2 Go1DribbleTest task.

File: assets/urdf/go1/urdf/go1-visual-backup.urdf (robot description, URDF)
Before this commit: robot go1_description, 23 links, 22 joints
Links:
- link FL_calf: geometry collision box size=0.213 0.016 0.016; visual mesh filename=../meshes/calf.stl scale=1 1 1
- link FL_foot: geometry collision sphere radius=0.02; visual sphere radius=0.01
- link FL_hip: geometry collision cylinder length=0.04 radius=0.046; visual mesh filename=../meshes/hip.stl scale=1 1 1
- link FL_thigh: geometry collision box size=0.213 0.0245 0.034; visual mesh filename=../meshes/thigh.stl scale=1 1 1
- link FR_calf: geometry collision box size=0.213 0.016 0.016; visual mesh filename=../meshes/calf.stl scale=1 1 1
- link FR_foot: geometry collision sphere radius=0.02; visual sphere radius=0.01
- link FR_hip: geometry collision cylinder length=0.04 radius=0.046; visual mesh filename=../meshes/hip.stl scale=1 1 1
- link FR_thigh: geometry collision box size=0.213 0.0245 0.034; visual mesh filename=../meshes/thigh_mirror.stl scale=1 1 1
- link RL_calf: geometry collision box size=0.213 0.016 0.016; visual mesh filename=../meshes/calf.stl scale=1 1 1
- link RL_foot: geometry collision sphere radius=0.02; visual sphere radius=0.01
- link RL_hip: geometry collision cylinder length=0.04 radius=0.046; visual mesh filename=../meshes/hip.stl scale=1 1 1
- link RL_thigh: geometry collision box size=0.213 0.0245 0.034; visual mesh filename=../meshes/thigh.stl scale=1 1 1
- link RR_calf: geometry collision box size=0.213 0.016 0.016; visual mesh filename=../meshes/calf.stl scale=1 1 1
- link RR_foot: geometry collision sphere radius=0.02; visual sphere radius=0.01
- link RR_hip: geometry collision cylinder length=0.04 radius=0.046; visual mesh filename=../meshes/hip.stl scale=1 1 1
- link RR_thigh: geometry collision box size=0.213 0.0245 0.034; visual mesh filename=../meshes/thigh_mirror.stl scale=1 1 1
- link base: geometry visual box size=0.001 0.001 0.001
- link imu_link: geometry visual box size=0.001 0.001 0.001
- link trunk: geometry collision box size=0.3762 0.0935 0.114; visual mesh filename=../meshes/trunk.stl scale=1 1 1
